File: Power_Board_EU/Power_Board_EU.sch (KiCad schematic (older format))
At the start: 13 parts

Commit message: Fixed all connections on ROFL
Parts:
- added C? (x2): 100nF, symbol C
- added J?: USB, symbol USB
- added P?: CONN_6, symbol CONN_6
- added P? (x2): CONN_2, symbol CONN_2
- added P?: CONN_8, symbol CONN_8
Connections:
- net labels added: D+, D-, RXD, TXD
- wire segments 27 -> 49
- no-connect marks 12 -> 13
Other:
- note added: "CBUS"
- note added: "External Supply"
Changed lines of the file:
@@
-EESchema Schematic File Version 2  date Mon 16 Apr 2012 02:08:39 PM EDT
+EESchema Schematic File Version 2  date Mon 30 Apr 2012 01:35:04 PM EDT
 LIBS:power
 LIBS:device
@@
 Sheet 1 1
 Title "Power Board EU version"
-Date "16 apr 2012"
+Date "30 apr 2012"
 Rev "0"
 Comp "I Heart Engineering"
@@
 Text Label 5050 1650 0    60   ~ 0
 5V
-NoConn ~ 5050 2900
 $Comp
 L CONN_2 P?
@@
 	1    0    0    -1
 $EndComp
-Wire Wire Line
-	2550 3800 2550 3600
-Wire Wire Line
-	2600 2500 2600 2350
-Wire Wire Line
-	3150 2900 4000 2900
-Connection ~ 3650 2900
-Wire Wire Line
-	3200 1650 4000 1650
-Connection ~ 3650 1650
-Wire Wire Line
-	3650 3800 3650 3300
-Wire Wire Line
-	4000 3300 4000 3800
-Wire Wire Line
-	4000 2500 4000 2050
-Wire Wire Line
-	3650 2050 3650 2500
-Wire Wire Line
-	1650 2050 1650 2500
-Wire Wire Line
-	1650 3300 1650 3750
-Wire Wire Line
-	1950 2900 1300 2900
-Wire Wire Line
-	2000 1650 1650 1650
-Wire Wire Line
-	1300 3750 1300 3350
-Wire Wire Line
-	1300 2900 1300 2950
-Connection ~ 1650 2900
-Wire Wire Line
-	1950 3150 1900 3150
-Wire Wire Line
-	1900 3150 1900 2900
-Connection ~ 1900 2900
-Wire Wire Line
-	2000 1900 1950 1900
-Wire Wire Line
-	1950 1900 1950 1650
-Connection ~ 1950 1650
-Wire Wire Line
-	6000 3600 6000 3900
-Wire Wire Line
-	6150 3600 6150 3800
-Wire Wire Line
-	5700 3800 6300 3800
-Connection ~ 6000 3800
-Wire Wire Line
-	5850 3800 5850 3600
-Wire Wire Line
-	5700 3800 5700 3600
-Connection ~ 5850 3800
-Wire Wire Line
-	6300 3800 6300 3600
-Connection ~ 6150 3800
-Wire Wire Line
-	8800 2450 8800 2600
 $Comp
 L CONN_2 P?
@@
 	1    0    0    -1
 $EndComp
-Wire Wire Line
-	8800 1900 8800 2050
 $Comp
 L CONN_2 P?
@@
 	1    0    0    -1
 $EndComp
-Wire Wire Line
-	9650 2450 9650 2600
 Text Label 9650 2250 0    60   ~ 0
 5V
@@
 Text Notes 8850 2850 0    60   ~ 0
 OUTPUT
-Text Notes 2900 5000 0    60   ~ 0
+Text Notes 3150 4950 0    60   ~ 0
 TO ROOMBA
-Text Notes 4500 5000 0    60   ~ 0
+Text Notes 4900 4500 0    60   ~ 0
 TO USB
+$Comp
+L CONN_6 P?
+U 1 1 4F9EC434
+P 7550 2750
+F 0 "P?" V 7500 2750 60  0000 C CNN
+F 1 "CONN_6" V 7600 2750 60  0000 C CNN
+	1    7550 2750
+	1    0    0    -1
+$EndComp
+$Comp
+L GND #PWR?
+U 1 1 4F9EC44E
+P 7200 3150
+F 0 "#PWR?" H 7200 3150 30  0001 C CNN
+F 1 "GND" H 7200 3080 30  0001 C CNN
+	1    7200 3150
+	1    0    0    -1
+$EndComp
+Text Label 7200 3000 2    60   ~ 0
+GND
+Text Notes 7650 2400 2    60   ~ 0
+CBUS
+$Comp
+L C C?
+U 1 1 4F9EC711
+P 5050 3200
+F 0 "C?" H 5100 3300 50  0000 L CNN
+F 1 "100nF" H 5100 3100 50  0000 L CNN
+	1    5050 3200
+	1    0    0    -1
+$EndComp
+$Comp
+L GND #PWR?
+U 1 1 4F9EC717
+P 5050 3900
+F 0 "#PWR?" H 5050 3900 30  0001 C CNN
+F 1 "GND" H 5050 3830 30  0001 C CNN
+	1    5050 3900
+	1    0    0    -1
+$EndComp
+$Comp
+L C C?
+U 1 1 4F9EC731
+P 4700 1850
+F 0 "C?" H 4750 1950 50  0000 L CNN
+F 1 "100nF" H 4750 1750 50  0000 L CNN
+	1    4700 1850
+	1    0    0    -1
+$EndComp
+$Comp
+L GND #PWR?
+U 1 1 4F9EC737
+P 4700 2550
+F 0 "#PWR?" H 4700 2550 30  0001 C CNN
+F 1 "GND" H 4700 2480 30  0001 C CNN
+	1    4700 2550
+	1    0    0    -1
+$EndComp
+$Comp
+L CONN_2 P?
+U 1 1 4F9EC865
+P 9300 1800
+F 0 "P?" V 9250 1800 40  0000 C CNN
+F 1 "CONN_2" V 9350 1800 40  0000 C CNN
+	1    9300 1800
+	-1   0    0    1
+$EndComp
+$Comp
+L GND #PWR?
+U 1 1 4F9EC86B
+P 9650 2050
+F 0 "#PWR?" H 9650 2050 30  0001 C CNN
+F 1 "GND" H 9650 1980 30  0001 C CNN
+	1    9650 2050
+	1    0    0    -1
+$EndComp
+Text Label 9650 1700 0    60   ~ 0
+5V
+$Comp
+L CONN_2 P?
+U 1 1 4F9EC873
+P 8250 3450
+F 0 "P?" V 8200 3450 40  0000 C CNN
+F 1 "CONN_2" V 8300 3450 40  0000 C CNN
+	1    8250 3450
+	-1   0    0    1
+$EndComp
+$Comp
+L GND #PWR?
+U 1 1 4F9EC879
+P 8600 3700
+F 0 "#PWR?" H 8600 3700 30  0001 C CNN
+F 1 "GND" H 8600 3630 30  0001 C CNN
+	1    8600 3700
+	1    0    0    -1
+$EndComp
+Text Label 8600 3350 0    60   ~ 0
+V_BAT
+Text Notes 8850 3200 2    60   ~ 0
+External Supply
+$Comp
+L CONN_8 P?
+U 1 1 4F9EC8FC
+P 3400 4450
+F 0 "P?" V 3350 4450 60  0000 C CNN
+F 1 "CONN_8" V 3450 4450 60  0000 C CNN
+	1    3400 4450
+	1    0    0    -1
+$EndComp
+$Comp
+L GND #PWR?
+U 1 1 4F9EC90D
+P 2950 4950
+F 0 "#PWR?" H 2950 4950 30  0001 C CNN
+F 1 "GND" H 2950 4880 30  0001 C CNN
+	1    2950 4950
+	1    0    0    -1
+$EndComp
+Text Label 2950 4100 2    60   ~ 0
+V_BAT
+Text Label 3050 4300 2    60   ~ 0
+TXD
+Text Label 3050 4400 2    60   ~ 0
+RXD
+NoConn ~ 3050 4500
+NoConn ~ 3050 4600
+Text Label 6900 1700 0    60   ~ 0
+TXD
+Text Label 6900 1800 0    60   ~ 0
+RXD
+$Comp
+L USB J?
+U 1 1 4F9ECAD6
+P 5650 4500
+F 0 "J?" H 5600 4900 60  0000 C CNN
+F 1 "USB" V 5400 4650 60  0000 C CNN
+	1    5650 4500
+	1    0    0    -1
+$EndComp
+$Comp
+L GND #PWR?
+U 1 1 4F9ECAE7
+P 5650 5200
+F 0 "#PWR?" H 5650 5200 30  0001 C CNN
+F 1 "GND" H 5650 5130 30  0001 C CNN
+	1    5650 5200
+	1    0    0    -1
+$EndComp
+Wire Wire Line
+	2550 3800 2550 3600
+Wire Wire Line
+	2600 2500 2600 2350
+Wire Wire Line
+	3150 2900 4000 2900
+Connection ~ 3650 2900
+Wire Wire Line
+	3200 1650 4000 1650
+Connection ~ 3650 1650
+Wire Wire Line
+	3650 3800 3650 3300
+Wire Wire Line
+	4000 3300 4000 3800
+Wire Wire Line
+	4000 2500 4000 2050
+Wire Wire Line
+	3650 2050 3650 2500
+Wire Wire Line
+	1650 2050 1650 2500
+Wire Wire Line
+	1650 3300 1650 3750
+Wire Wire Line
+	1950 2900 1300 2900
+Wire Wire Line
+	2000 1650 1650 1650
+Wire Wire Line
+	1300 3750 1300 3350
+Wire Wire Line
+	1300 2900 1300 2950
+Connection ~ 1650 2900
+Wire Wire Line
+	1950 3150 1900 3150
+Wire Wire Line
+	1900 3150 1900 2900
+Connection ~ 1900 2900
+Wire Wire Line
+	2000 1900 1950 1900
+Wire Wire Line
+	1950 1900 1950 1650
+Connection ~ 1950 1650
+Wire Wire Line
+	6000 3600 6000 3900
+Wire Wire Line
+	6150 3600 6150 3800
+Wire Wire Line
+	5700 3800 6300 3800
+Connection ~ 6000 3800
+Wire Wire Line
+	5850 3800 5850 3600
+Wire Wire Line
+	5700 3800 5700 3600
+Connection ~ 5850 3800
+Wire Wire Line
+	6300 3800 6300 3600
+Connection ~ 6150 3800
+Wire Wire Line
+	8800 2450 8800 2600
+Wire Wire Line
+	8800 1900 8800 2050
+Wire Wire Line
+	9650 2450 9650 2600
+Wire Wire Line
+	7200 2900 6900 2900
+Wire Wire Line
+	6900 2800 7200 2800
+Wire Wire Line
+	7200 2700 6900 2700
+Wire Wire Line
+	6900 2600 7200 2600
+Wire Wire Line
+	7200 2500 6900 2500
+Wire Wire Line
+	7200 3150 7200 3000
+Wire Wire Line
+	5050 3400 5050 3900
+Wire Wire Line
+	4700 2050 4700 2550
+Wire Wire Line
+	5050 1650 4700 1650
+Wire Wire Line
+	5050 2900 5050 3000
+Wire Wire Line
+	9650 1900 9650 2050
+Wire Wire Line
+	8600 3550 8600 3700
+Wire Wire Line
+	3050 4700 2950 4700
+Wire Wire Line
+	2950 4700 2950 4950
+Wire Wire Line
+	3050 4800 2950 4800
+Connection ~ 2950 4800
+Wire Wire Line
+	3050 4200 2950 4200
+Wire Wire Line
+	2950 4200 2950 4100
+Wire Wire Line
+	2950 4100 3050 4100
+Wire Wire Line
+	5650 5200 5650 5100
+Wire Wire Line
+	6000 4950 6000 5100
+Wire Wire Line
+	5250 5100 6000 5100
+Wire Wire Line
+	5250 4850 5250 5100
+Connection ~ 5650 5100
+Connection ~ 5250 4950
+Connection ~ 5250 4950
+Text Label 5250 4700 2    60   ~ 0
+5V
+Text Label 5050 2000 2    60   ~ 0
+D-
+Text Label 5050 2100 2    60   ~ 0
+D+
+Text Label 6000 4700 0    60   ~ 0
+D+
+Text Label 6000 4850 0    60   ~ 0
+D-
 $EndSCHEMATC

Commit message: Generated Gerber files EU Power Supply
Parts:
- added K1: CONN_3, symbol CONN_3
- gave numbers to parts that had none: 20
Connections:
- net labels added: V_EXT, V_IN
Other:
- note added: "Power Selector"

Commit message: Created Gerber files for Buttons Shield
Parts:
- added JMP1, JMP2: SJMP, symbol SJMP
- added P10, P9: CONN_8, symbol CONN_8
- added P11, P12: CONN_1, symbol CONN_1
- added P8: CONN_6, symbol CONN_6
- added SHIELD?: ARDUINO_MEGA_SHIELD, symbol ARDUINO_MEGA_SHIELD
- added SW1: SW_PUSH_SMALL, symbol SW_PUSH_SMALL
Connections:
- net labels added: EN12, EN5
- wire segments 49 -> 79
Other:
- moved on the sheet: C1, C2, C3, C4, C5, C6, D1, VR1, VR2

Commit message: Updated to Arduino Mega Shield
Parts:
- removed P8: CONN_6, symbol CONN_6
- added P15, P16, P17: CONN_8, symbol CONN_8
- gave numbers to parts that had none: 1
Connections:
- wire segments 79 -> 100
- no-connect marks 13 -> 49
Other:
- moved on the sheet: SHIELD1, SW1

Commit message: rearranged European Power Board
Parts:
- removed D1: DIODE, symbol DIODE
- removed P2: CONN_6, symbol CONN_6
Connections:
- wire segments 100 -> 90
- no-connect marks 49 -> 54
Other:
- note removed: "CBUS"
Changed lines of the file:
@@
-EESchema Schematic File Version 2  date Wed 30 May 2012 12:32:51 PM EDT
+EESchema Schematic File Version 2  date Mon 04 Jun 2012 06:28:09 PM EDT
 LIBS:power
 LIBS:device
@@
 Sheet 1 1
 Title "Power Board EU version"
-Date "30 may 2012"
+Date "4 jun 2012"
 Rev "0"
 Comp "I Heart Engineering"
@@
 F 1 "GND" H 8100 5880 30  0001 C CNN
 	1    8100 5950
-	1    0    0    -1
-$EndComp
-$Comp
-L DIODE D1
-U 1 1 4F8C5CCA
-P 7750 5350
-F 0 "D1" H 7750 5450 40  0000 C CNN
-F 1 "DIODE" H 7750 5250 40  0000 C CNN
-	1    7750 5350
-	0    -1   -1   0
-$EndComp
-$Comp
-L GND #PWR10
-U 1 1 4F8C5CD7
-P 7750 5950
-F 0 "#PWR10" H 7750 5950 30  0001 C CNN
-F 1 "GND" H 7750 5880 30  0001 C CNN
-	1    7750 5950
 	1    0    0    -1
 $EndComp
@@
 Text Notes 4900 4500 0    60   ~ 0
 TO USB
-$Comp
-L CONN_6 P2
-U 1 1 4F9EC434
-P 7550 2750
-F 0 "P2" V 7500 2750 60  0000 C CNN
-F 1 "CONN_6" V 7600 2750 60  0000 C CNN
-	1    7550 2750
-	1    0    0    -1
-$EndComp
-$Comp
-L GND #PWR9
-U 1 1 4F9EC44E
-P 7200 3150
-F 0 "#PWR9" H 7200 3150 30  0001 C CNN
-F 1 "GND" H 7200 3080 30  0001 C CNN
-	1    7200 3150
-	1    0    0    -1
-$EndComp
-Text Label 7200 3000 2    60   ~ 0
-GND
-Text Notes 7650 2400 2    60   ~ 0
-CBUS
 $Comp
 L C C8
@@
 	0    -1   -1   0
 $EndComp
+Text Label 4150 3150 2    60   ~ 0
+5V
+Text Label 4150 3550 2    60   ~ 0
+5V
 Wire Wire Line
 	9000 6000 9000 5800
@@
 	8100 5500 8100 5950
 Wire Wire Line
-	7750 5100 8400 5100
-Wire Wire Line
 	8100 3850 8450 3850
-Wire Wire Line
-	7750 5950 7750 5550
-Wire Wire Line
-	7750 5100 7750 5150
 Connection ~ 8100 5100
 Wire Wire Line
 	8400 5350 8400 5650
-Connection ~ 8350 5100
 Wire Wire Line
 	8450 4100 8450 4350
@@
 Wire Wire Line
 	9650 2450 9650 2600
-Wire Wire Line
-	7200 2900 6900 2900
-Wire Wire Line
-	6900 2800 7200 2800
-Wire Wire Line
-	7200 2700 6900 2700
-Wire Wire Line
-	6900 2600 7200 2600
-Wire Wire Line
-	7200 2500 6900 2500
-Wire Wire Line
-	7200 3150 7200 3000
 Wire Wire Line
 	5050 3400 5050 3900
@@
 Connection ~ 1200 5350
 Wire Wire Line
-	3350 3600 4150 3150
-Connection ~ 3350 3600
-Connection ~ 3350 3600
-Wire Wire Line
-	3350 3700 4150 3550
-Connection ~ 3350 3700
-Connection ~ 3350 3700
+	8100 5100 8400 5100
+NoConn ~ 6900 2500
+NoConn ~ 6900 2600
+NoConn ~ 6900 2700
+NoConn ~ 6900 2800
+NoConn ~ 6900 2900
 $EndSCHEMATC

Commit message: Added Snap conn Button Shield
Parts:
- removed JMP1, JMP2: SJMP, symbol SJMP
- removed P1, P10, P15, P16, P17, P9: CONN_8, symbol CONN_8
- removed P11, P12: CONN_1, symbol CONN_1
- added K1: CONN_3, symbol CONN_3
- added P6: CONN_7, symbol CONN_7
- added R1, R2: 10k, symbol R
- added SW2: DPDT, symbol DPDT
- added SW3: SWITCH_INV, symbol SWITCH_INV
- renumbered C7 to C1, C8 to C2, C1 to C3, C2 to C4, C3 to C5, C4 to C6, C5 to C7, C6 to C8, K1 to K2, P6 to P10, P7 to P11, P3 to P7, P4 to P8, P5 to P9
Connections:
- net labels added: 5V_FTDI, 5V_USB, D6, D7
- wire segments 90 -> 52
- no-connect marks 54 -> 88
Other:
- note added: "FTDI Chip Power Selector"
- note added: "Voltage Regulator Enabler"
- moved on the sheet: K2

Commit message: Finished Gerbers for Button Shield
Parts:
- renumbered P6 to P1, P7 to P2, P8 to P3, P9 to P4, P10 to P5, P11 to P6
Changed lines of the file:
@@
-EESchema Schematic File Version 2  date Wed 06 Jun 2012 03:27:17 PM EDT
+EESchema Schematic File Version 2  date Wed 06 Jun 2012 08:03:03 PM EDT
 LIBS:power
 LIBS:device
@@
 $EndComp
 $Comp
-L GND #PWR01
+L GND #PWR16
 U 1 1 4F8C5B26
 P 9000 6000
-F 0 "#PWR01" H 9000 6000 30  0001 C CNN
+F 0 "#PWR16" H 9000 6000 30  0001 C CNN
 F 1 "GND" H 9000 5930 30  0001 C CNN
 	1    9000 6000
@@
 $EndComp
 $Comp
-L GND #PWR02
+L GND #PWR17
 U 1 1 4F8C5B35
 P 9050 4700
-F 0 "#PWR02" H 9050 4700 30  0001 C CNN
+F 0 "#PWR17" H 9050 4700 30  0001 C CNN
 F 1 "GND" H 9050 4630 30  0001 C CNN
 	1    9050 4700
@@
 $EndComp
 $Comp
-L GND #PWR03
+L GND #PWR22
 U 1 1 4F8C5BC4
 P 10450 4700
-F 0 "#PWR03" H 10450 4700 30  0001 C CNN
+F 0 "#PWR22" H 10450 4700 30  0001 C CNN
 F 1 "GND" H 10450 4630 30  0001 C CNN
 	1    10450 4700
@@
 $EndComp
 $Comp
-L GND #PWR04
+L GND #PWR20
 U 1 1 4F8C5BD1
 P 10100 4700
-F 0 "#PWR04" H 10100 4700 30  0001 C CNN
+F 0 "#PWR20" H 10100 4700 30  0001 C CNN
 F 1 "GND" H 10100 4630 30  0001 C CNN
 	1    10100 4700
@@
 $EndComp
 $Comp
-L GND #PWR05
+L GND #PWR23
 U 1 1 4F8C5BD7
 P 10450 6000
-F 0 "#PWR05" H 10450 6000 30  0001 C CNN
+F 0 "#PWR23" H 10450 6000 30  0001 C CNN
 F 1 "GND" H 10450 5930 30  0001 C CNN
 	1    10450 6000
@@
 $EndComp
 $Comp
-L GND #PWR06
+L GND #PWR21
 U 1 1 4F8C5BDD
 P 10100 6000
-F 0 "#PWR06" H 10100 6000 30  0001 C CNN
+F 0 "#PWR21" H 10100 6000 30  0001 C CNN
 F 1 "GND" H 10100 5930 30  0001 C CNN
 	1    10100 6000
@@
 $EndComp
 $Comp
-L GND #PWR07
+L GND #PWR11
 U 1 1 4F8C5C56
 P 8100 4700
-F 0 "#PWR07" H 8100 4700 30  0001 C CNN
+F 0 "#PWR11" H 8100 4700 30  0001 C CNN
 F 1 "GND" H 8100 4630 30  0001 C CNN
 	1    8100 4700
@@
 $EndComp
 $Comp
-L GND #PWR08
+L GND #PWR12
 U 1 1 4F8C5C63
 P 8100 5950
-F 0 "#PWR08" H 8100 5950 30  0001 C CNN
+F 0 "#PWR12" H 8100 5950 30  0001 C CNN
 F 1 "GND" H 8100 5880 30  0001 C CNN
 	1    8100 5950
@@
 $EndComp
 $Comp
-L GND #PWR09
+L GND #PWR9
 U 1 1 4F8C5F75
 P 6000 3900
-F 0 "#PWR09" H 6000 3900 30  0001 C CNN
+F 0 "#PWR9" H 6000 3900 30  0001 C CNN
 F 1 "GND" H 6000 3830 30  0001 C CNN
 	1    6000 3900
@@
 5V_FTDI
 $Comp
-L CONN_2 P9
+L CONN_2 P4
 U 1 1 4F8C62BB
 P 8450 2350
-F 0 "P9" V 8400 2350 40  0000 C CNN
+F 0 "P4" V 8400 2350 40  0000 C CNN
 F 1 "CONN_2" V 8500 2350 40  0000 C CNN
 	1    8450 2350
@@
 $EndComp
 $Comp
-L GND #PWR010
+L GND #PWR15
 U 1 1 4F8C62D4
 P 8800 2600
-F 0 "#PWR010" H 8800 2600 30  0001 C CNN
+F 0 "#PWR15" H 8800 2600 30  0001 C CNN
 F 1 "GND" H 8800 2530 30  0001 C CNN
 	1    8800 2600
@@
 $EndComp
 $Comp
-L CONN_2 P8
+L CONN_2 P3
 U 1 1 4F8C6322
 P 8450 1800
-F 0 "P8" V 8400 1800 40  0000 C CNN
+F 0 "P3" V 8400 1800 40  0000 C CNN
 F 1 "CONN_2" V 8500 1800 40  0000 C CNN
 	1    8450 1800
@@
 $EndComp
 $Comp
-L GND #PWR011
+L GND #PWR14
 U 1 1 4F8C6328
 P 8800 2050
-F 0 "#PWR011" H 8800 2050 30  0001 C CNN
+F 0 "#PWR14" H 8800 2050 30  0001 C CNN
 F 1 "GND" H 8800 1980 30  0001 C CNN
 	1    8800 2050
@@
 $EndComp
 $Comp
-L CONN_2 P11
+L CONN_2 P6
 U 1 1 4F8C632F
 P 9300 2350
-F 0 "P11" V 9250 2350 40  0000 C CNN
+F 0 "P6" V 9250 2350 40  0000 C CNN
 F 1 "CONN_2" V 9350 2350 40  0000 C CNN
 	1    9300 2350
@@
 $EndComp
 $Comp
-L GND #PWR012
+L GND #PWR19
 U 1 1 4F8C6335
 P 9650 2600
-F 0 "#PWR012" H 9650 2600 30  0001 C CNN
+F 0 "#PWR19" H 9650 2600 30  0001 C CNN
 F 1 "GND" H 9650 2530 30  0001 C CNN
 	1    9650 2600
@@
 $EndComp
 $Comp
-L GND #PWR013
+L GND #PWR6
 U 1 1 4F9EC717
 P 5050 3900
-F 0 "#PWR013" H 5050 3900 30  0001 C CNN
+F 0 "#PWR6" H 5050 3900 30  0001 C CNN
 F 1 "GND" H 5050 3830 30  0001 C CNN
 	1    5050 3900
@@
 $EndComp
 $Comp
-L GND #PWR014
+L GND #PWR4
 U 1 1 4F9EC737
 P 4700 2550
-F 0 "#PWR014" H 4700 2550 30  0001 C CNN
+F 0 "#PWR4" H 4700 2550 30  0001 C CNN
 F 1 "GND" H 4700 2480 30  0001 C CNN
 	1    4700 2550
@@
 $EndComp
 $Comp
-L CONN_2 P10
+L CONN_2 P5
 U 1 1 4F9EC865
 P 9300 1800
-F 0 "P10" V 9250 1800 40  0000 C CNN
+F 0 "P5" V 9250 1800 40  0000 C CNN
 F 1 "CONN_2" V 9350 1800 40  0000 C CNN
 	1    9300 1800
@@
 $EndComp
 $Comp
-L GND #PWR015
+L GND #PWR18
 U 1 1 4F9EC86B
 P 9650 2050
-F 0 "#PWR015" H 9650 2050 30  0001 C CNN
+F 0 "#PWR18" H 9650 2050 30  0001 C CNN
 F 1 "GND" H 9650 1980 30  0001 C CNN
 	1    9650 2050
@@
 5V
 $Comp
-L CONN_2 P7
+L CONN_2 P2
 U 1 1 4F9EC873
 P 8250 3450
-F 0 "P7" V 8200 3450 40  0000 C CNN
+F 0 "P2" V 8200 3450 40  0000 C CNN
 F 1 "CONN_2" V 8300 3450 40  0000 C CNN
 	1    8250 3450
@@
 $EndComp
 $Comp
-L GND #PWR016
+L GND #PWR13
 U 1 1 4F9EC879
 P 8600 3700
-F 0 "#PWR016" H 8600 3700 30  0001 C CNN
+F 0 "#PWR13" H 8600 3700 30  0001 C CNN
 F 1 "GND" H 8600 3630 30  0001 C CNN
 	1    8600 3700
@@
 External Supply
 $Comp
-L GND #PWR017
+L GND #PWR10
 U 1 1 4F9EC90D
 P 6650 4950
-F 0 "#PWR017" H 6650 4950 30  0001 C CNN
+F 0 "#PWR10" H 6650 4950 30  0001 C CNN
 F 1 "GND" H 6650 4880 30  0001 C CNN
 	1    6650 4950
@@
 $EndComp
 $Comp
-L GND #PWR018
+L GND #PWR8
 U 1 1 4F9ECAE7
 P 5650 5200
-F 0 "#PWR018" H 5650 5200 30  0001 C CNN
+F 0 "#PWR8" H 5650 5200 30  0001 C CNN
 F 1 "GND" H 5650 5130 30  0001 C CNN
 	1    5650 5200
@@
 V_EXT
 $Comp
-L GND #PWR019
+L GND #PWR2
 U 1 1 4FC532E3
 P 1100 3150
-F 0 "#PWR019" H 1100 3150 30  0001 C CNN
+F 0 "#PWR2" H 1100 3150 30  0001 C CNN
 F 1 "GND" H 1100 3080 30  0001 C CNN
 	1    1100 3150
@@
 $EndComp
 $Comp
-L GND #PWR020
+L GND #PWR1
 U 1 1 4FC54E9D
 P 590 2580
-F 0 "#PWR020" H 590 2580 30  0001 C CNN
+F 0 "#PWR1" H 590 2580 30  0001 C CNN
 F 1 "GND" H 590 2510 30  0001 C CNN
 	1    590  2580
@@
 $EndComp
 $Comp
-L GND #PWR021
+L GND #PWR3
 U 1 1 4FC658D8
 P 1200 5400
-F 0 "#PWR021" H 1200 5400 30  0001 C CNN
+F 0 "#PWR3" H 1200 5400 30  0001 C CNN
 F 1 "GND" H 1200 5330 30  0001 C CNN
 	1    1200 5400
@@
 FTDI Chip Power Selector
 $Comp
-L GND #PWR022
+L GND #PWR5
 U 1 1 4FCF76FF
 P 4850 6900
-F 0 "#PWR022" H 4850 6900 30  0001 C CNN
+F 0 "#PWR5" H 4850 6900 30  0001 C CNN
 F 1 "GND" H 4850 6830 30  0001 C CNN
 	1    4850 6900
@@
 $EndComp
 $Comp
-L GND #PWR023
+L GND #PWR7
 U 1 1 4FCF770E
 P 5250 6450
-F 0 "#PWR023" H 5250 6450 30  0001 C CNN
+F 0 "#PWR7" H 5250 6450 30  0001 C CNN
 F 1 "GND" H 5250 6380 30  0001 C CNN
 	1    5250 6450
@@
 $EndComp
 $Comp
-L CONN_7 P6
+L CONN_7 P1
 U 1 1 4FCF7A45
 P 7100 4500
-F 0 "P6" V 7070 4500 60  0000 C CNN
+F 0 "P1" V 7070 4500 60  0000 C CNN
 F 1 "CONN_7" V 7170 4500 60  0000 C CNN
 	1    7100 4500
