File: RingOfFireLight/RingOfFireLight.sch (KiCad schematic (older format))
At the start: 43 parts

Commit message: Added board file
Parts:
- removed P? (x2): CONN_5, symbol CONN_5
- added P1, P2: CONN_6, symbol CONN_6
- added P3: CONN_2, symbol CONN_2
- gave numbers to parts that had none: 41
Connections:
- net V_LED is gone; now on net 12V: C1.1, D1.1 (A), D10.1 (A), D11.1 (A), D12.1 (A), D13.1 (A), D14.1 (A), D15.1 (A), D16.1 (A), D2.1 (A), D3.1 (A), D4.1 (A), D5.1 (A), D6.1 (A), D7.1 (A), D8.1 (A), D9.1 (A), U1.1 (VIN), U1.3 (ON/OFF)
- net GND: now also P1.6, P2.6, P3.1 (P1)
- net GSCLK: now also P1.2, P2.2
- net MOSI: now also P2.1
- net SCK: now also R3.2, P1.3, P2.3
- net SOUT: now also P1.1
- net VCC: now also P1.4, P2.4
- net RAW renamed 12V
- net 12V: now also P1.5, P2.5, P3.2 (PM)
Other:
- note added: "ATMega328 \n32 TQFP"
- note added: "Board to board connectors"
- note added: "Power Connector"
- note removed: "look up board to board conn."
- note removed: "make sure to be able to plug the arduino mino pro and have everything work"
- moved on the sheet: C5

Commit message: Organized components
Parts:
- removed C6, C7: 22pF, symbol C
- removed X1: 16MHz, symbol CRYSTAL
- added X1: RESONATOR, symbol RESONATOR
Connections:
- wire segments 118 -> 116
Other:
- note added: "Resonator\n490-1198-1-ND"
Changed lines of the file:
@@
-EESchema Schematic File Version 2  date Mon 26 Mar 2012 01:38:16 PM EDT
+EESchema Schematic File Version 2  date Wed 28 Mar 2012 04:07:31 PM EDT
 LIBS:power
 LIBS:device
@@
 LIBS:valves
 LIBS:tlc5940
+LIBS:resonator
 LIBS:RingOfFireLight-cache
 EELAYER 25  0
@@
 Sheet 1 1
 Title "LED circle with Arduino Mini 328"
-Date "26 mar 2012"
+Date "28 mar 2012"
 Rev "0"
 Comp "I Heart Engineering"
@@
 $EndComp
 $Comp
-L CRYSTAL X1
-U 1 1 4F652C1E
-P 9450 6550
-F 0 "X1" V 9450 6700 60  0000 C CNN
-F 1 "16MHz" V 9450 6300 60  0000 C CNN
-	1    9450 6550
-	0    1    1    0
-$EndComp
-$Comp
-L C C7
-U 1 1 4F652C30
-P 9700 6850
-F 0 "C7" V 9750 6950 50  0000 L CNN
-F 1 "22pF" V 9550 6650 50  0000 L CNN
-	1    9700 6850
-	0    -1   -1   0
-$EndComp
-$Comp
-L C C6
-U 1 1 4F652C36
-P 9700 6250
-F 0 "C6" V 9750 6350 50  0000 L CNN
-F 1 "22pF" V 9750 6000 50  0000 L CNN
-	1    9700 6250
-	0    -1   -1   0
-$EndComp
-$Comp
 L GND #PWR09
 U 1 1 4F652CC7
-P 10200 6650
-F 0 "#PWR09" H 10200 6650 30  0001 C CNN
-F 1 "GND" H 10200 6580 30  0001 C CNN
-	1    10200 6650
+P 10000 6700
+F 0 "#PWR09" H 10000 6700 30  0001 C CNN
+F 1 "GND" H 10000 6630 30  0001 C CNN
+	1    10000 6700
 	1    0    0    -1
 $EndComp
@@
 Text Label 8000 5200 0    60   ~ 0
 TOSC2
-Text Label 9100 6850 0    60   ~ 0
+Text Label 8700 6800 0    60   ~ 0
 TOSC2
-Text Label 9100 6250 0    60   ~ 0
+Text Label 8700 6250 0    60   ~ 0
 TOSC1
 Text Label 9150 5000 0    60   ~ 0
@@
 Text Label 3850 4050 0    60   ~ 0
 V_LED
-Wire Wire Line
-	9500 6250 9100 6250
+Text Notes 9100 6900 0    60   ~ 0
+Resonator\n490-1198-1-ND
+Wire Wire Line
+	9100 6250 8700 6250
 Wire Wire Line
 	8000 5200 7850 5200
 Wire Wire Line
 	7850 5100 8000 5100
-Connection ~ 9450 6250
-Connection ~ 9450 6850
-Connection ~ 9900 6500
-Connection ~ 9900 6500
-Wire Wire Line
-	9900 6850 9900 6250
-Wire Wire Line
-	9900 6500 10200 6500
-Wire Wire Line
-	9500 6850 9100 6850
+Wire Wire Line
+	9100 6800 8700 6800
 Wire Wire Line
 	9650 4000 9650 3900
@@
 	6200 1100 4950 1100
 Wire Wire Line
-	10200 6500 10200 6650
-Wire Wire Line
 	4950 1100 4950 1200
 Wire Wire Line
@@
 Wire Wire Line
 	6200 2300 6200 2150
+Wire Wire Line
+	10000 6550 10000 6700
+$Comp
+L RESONATOR X1
+U 1 1 4F7370F4
+P 9400 6550
+F 0 "X1" H 9400 6700 60  0000 C CNN
+F 1 "RESONATOR" H 9400 6400 60  0000 C CNN
+	1    9400 6550
+	0    -1   -1   0
+$EndComp
 $EndSCHEMATC

Commit message: Layout Draft 1
Parts:
- removed P7: CONN_6, symbol CONN_6
- removed X1: RESONATOR, symbol RESONATOR
- added C6, C9: 0.1uF, symbol C
- added C7: 10uF 25V, symbol CP1
- added D19, D20: LED, symbol LED
- added J1: USB_2, symbol USB_2
- added R6, R7: 1k, symbol R
- added U2: FT232RL, symbol FT232RL
- added X1: XTAL_RESONATOR, symbol XTAL_RESONATOR
Connections:
- net labels added: POWER
- wire segments 116 -> 140
- no-connect marks 1 -> 11
Other:
- moved on the sheet: C1, C3, C4, D18, P3, R4, U1

Commit message: Updated BOM, Added Board-to-Board connectors
Parts:
- added K1: CONN_3, symbol CONN_3
Other:
- note added: "Arduino Pro Mini Connectors"
- note added: "Sensor Connectors"
- moved on the sheet: P4, P5, P6
Changed lines of the file:
@@
-EESchema Schematic File Version 2  date Mon 02 Apr 2012 07:08:28 PM EDT
+EESchema Schematic File Version 2  date Mon 09 Apr 2012 08:06:20 PM EDT
 LIBS:power
 LIBS:device
@@
 Sheet 1 1
 Title "LED circle with Arduino Mini 328"
-Date "2 apr 2012"
+Date "10 apr 2012"
 Rev "0"
 Comp "I Heart Engineering"
@@
 $EndComp
 $Comp
-L GND #PWR01
+L GND #PWR10
 U 1 1 4F650B60
 P 5800 6900
-F 0 "#PWR01" H 5800 6900 30  0001 C CNN
+F 0 "#PWR10" H 5800 6900 30  0001 C CNN
 F 1 "GND" H 5800 6830 30  0001 C CNN
 	1    5800 6900
@@
 $EndComp
 $Comp
-L VCC #PWR02
+L VCC #PWR9
 U 1 1 4F65226B
 P 5800 4250
-F 0 "#PWR02" H 5800 4350 30  0001 C CNN
+F 0 "#PWR9" H 5800 4350 30  0001 C CNN
 F 1 "VCC" H 5800 4350 30  0000 C CNN
 	1    5800 4250
@@
 $EndComp
 $Comp
-L GND #PWR03
+L GND #PWR8
 U 1 1 4F652516
 P 5700 5650
-F 0 "#PWR03" H 5700 5650 30  0001 C CNN
+F 0 "#PWR8" H 5700 5650 30  0001 C CNN
 F 1 "GND" H 5700 5580 30  0001 C CNN
 	1    5700 5650
@@
 $EndComp
 $Comp
-L GND #PWR04
+L GND #PWR13
 U 1 1 4F652546
 P 8500 6000
-F 0 "#PWR04" H 8500 6000 30  0001 C CNN
+F 0 "#PWR13" H 8500 6000 30  0001 C CNN
 F 1 "GND" H 8500 5930 30  0001 C CNN
 	1    8500 6000
@@
 $EndComp
 $Comp
-L VCC #PWR05
+L VCC #PWR15
 U 1 1 4F652713
 P 9500 4450
-F 0 "#PWR05" H 9500 4550 30  0001 C CNN
+F 0 "#PWR15" H 9500 4550 30  0001 C CNN
 F 1 "VCC" H 9500 4550 30  0000 C CNN
 	1    9500 4450
@@
 $EndComp
 $Comp
-L GND #PWR06
+L GND #PWR16
 U 1 1 4F65277D
 P 9500 5800
-F 0 "#PWR06" H 9500 5800 30  0001 C CNN
+F 0 "#PWR16" H 9500 5800 30  0001 C CNN
 F 1 "GND" H 9500 5730 30  0001 C CNN
 	1    9500 5800
@@
 $EndComp
 $Comp
-L VCC #PWR07
+L VCC #PWR19
 U 1 1 4F652AEC
 P 9650 3400
-F 0 "#PWR07" H 9650 3500 30  0001 C CNN
+F 0 "#PWR19" H 9650 3500 30  0001 C CNN
 F 1 "VCC" H 9650 3500 30  0000 C CNN
 	1    9650 3400
@@
 $EndComp
 $Comp
-L GND #PWR08
+L GND #PWR20
 U 1 1 4F652AFB
 P 9650 4000
-F 0 "#PWR08" H 9650 4000 30  0001 C CNN
+F 0 "#PWR20" H 9650 4000 30  0001 C CNN
 F 1 "GND" H 9650 3930 30  0001 C CNN
 	1    9650 4000
@@
 $EndComp
 $Comp
-L GND #PWR09
+L GND #PWR21
 U 1 1 4F652CC7
 P 9900 6650
-F 0 "#PWR09" H 9900 6650 30  0001 C CNN
+F 0 "#PWR21" H 9900 6650 30  0001 C CNN
 F 1 "GND" H 9900 6580 30  0001 C CNN
 	1    9900 6650
@@
 L CONN_12 P5
 U 1 1 4F65EEDB
-P 7100 3450
-F 0 "P5" V 7050 3450 60  0000 C CNN
-F 1 "CONN_12" V 7150 3450 60  0000 C CNN
-	1    7100 3450
+P 7450 3450
+F 0 "P5" V 7400 3450 60  0000 C CNN
+F 1 "CONN_12" V 7500 3450 60  0000 C CNN
+	1    7450 3450
 	-1   0    0    1
 $EndComp
@@
 L CONN_12 P4
 U 1 1 4F65EF1D
-P 6150 3450
-F 0 "P4" V 6100 3450 60  0000 C CNN
-F 1 "CONN_12" V 6200 3450 60  0000 C CNN
-	1    6150 3450
+P 6500 3450
+F 0 "P4" V 6450 3450 60  0000 C CNN
+F 1 "CONN_12" V 6550 3450 60  0000 C CNN
+	1    6500 3450
 	-1   0    0    1
 $EndComp
@@
 L CONN_2 P6
 U 1 1 4F65FCCB
-P 8000 3000
-F 0 "P6" V 7950 3000 40  0000 C CNN
-F 1 "CONN_2" V 8050 3000 40  0000 C CNN
-	1    8000 3000
+P 8350 3000
+F 0 "P6" V 8300 3000 40  0000 C CNN
+F 1 "CONN_2" V 8400 3000 40  0000 C CNN
+	1    8350 3000
 	-1   0    0    1
 $EndComp
@@
 Text Label 8000 4700 0    60   ~ 0
 D10
-Text Label 6500 2900 0    60   ~ 0
+Text Label 6850 2900 0    60   ~ 0
 TX
-Text Label 6500 3000 0    60   ~ 0
+Text Label 6850 3000 0    60   ~ 0
 RX
-Text Label 6500 3100 0    60   ~ 0
+Text Label 6850 3100 0    60   ~ 0
 RESET
-Text Label 6500 3200 0    60   ~ 0
+Text Label 6850 3200 0    60   ~ 0
 GND
 Text Label 9650 3950 0    60   ~ 0
@@
 Text Label 9650 3450 0    60   ~ 0
 VCC
-Text Label 6500 3300 0    60   ~ 0
+Text Label 6850 3300 0    60   ~ 0
 D2
-Text Label 6500 3400 0    60   ~ 0
+Text Label 6850 3400 0    60   ~ 0
 D3
-Text Label 6500 3500 0    60   ~ 0
+Text Label 6850 3500 0    60   ~ 0
 D4
-Text Label 6500 3600 0    60   ~ 0
+Text Label 6850 3600 0    60   ~ 0
 D5
-Text Label 6500 3700 0    60   ~ 0
+Text Label 6850 3700 0    60   ~ 0
 D6
-Text Label 6500 3800 0    60   ~ 0
+Text Label 6850 3800 0    60   ~ 0
 D7
-Text Label 6500 3900 0    60   ~ 0
+Text Label 6850 3900 0    60   ~ 0
 D8
-Text Label 6500 4000 0    60   ~ 0
+Text Label 6850 4000 0    60   ~ 0
 D9
-Text Label 7450 3000 0    60   ~ 0
+Text Label 7800 3000 0    60   ~ 0
 GND
-Text Label 7450 3100 0    60   ~ 0
+Text Label 7800 3100 0    60   ~ 0
 RESET
-Text Label 7450 3200 0    60   ~ 0
+Text Label 7800 3200 0    60   ~ 0
 VCC
-Text Label 7450 3300 0    60   ~ 0
+Text Label 7800 3300 0    60   ~ 0
 A3
-Text Label 7450 3400 0    60   ~ 0
+Text Label 7800 3400 0    60   ~ 0
 A2
-Text Label 7450 3500 0    60   ~ 0
+Text Label 7800 3500 0    60   ~ 0
 A1
-Text Label 7450 3600 0    60   ~ 0
+Text Label 7800 3600 0    60   ~ 0
 A0
-Text Label 7450 3700 0    60   ~ 0
+Text Label 7800 3700 0    60   ~ 0
 SCK
-Text Label 7450 3800 0    60   ~ 0
+Text Label 7800 3800 0    60   ~ 0
 MISO
-Text Label 7450 3900 0    60   ~ 0
+Text Label 7800 3900 0    60   ~ 0
 MOSI
-Text Label 7450 4000 0    60   ~ 0
+Text Label 7800 4000 0    60   ~ 0
 D10
 Text Label 5800 4400 0    60   ~ 0
@@
 Text Label 3800 1800 0    60   ~ 0
 DTR
-Text Label 8350 2900 0    60   ~ 0
+Text Label 8700 2900 0    60   ~ 0
 A4
-Text Label 8350 3100 0    60   ~ 0
+Text Label 8700 3100 0    60   ~ 0
 A5
 $Comp
@@
 $EndComp
 $Comp
-L GND #PWR010
+L GND #PWR7
 U 1 1 4F66B442
 P 4600 6250
-F 0 "#PWR010" H 4600 6250 30  0001 C CNN
+F 0 "#PWR7" H 4600 6250 30  0001 C CNN
 F 1 "GND" H 4600 6180 30  0001 C CNN
 	1    4600 6250
@@
 $EndComp
 $Comp
-L VCC #PWR011
+L VCC #PWR6
 U 1 1 4F6745B5
 P 4550 5550
-F 0 "#PWR011" H 4550 5650 30  0001 C CNN
+F 0 "#PWR6" H 4550 5650 30  0001 C CNN
 F 1 "VCC" H 4550 5650 30  0000 C CNN
 	1    4550 5550
@@
 $EndComp
 $Comp
-L GND #PWR012
+L GND #PWR14
 U 1 1 4F69ECF8
 P 8600 2200
-F 0 "#PWR012" H 8600 2200 30  0001 C CNN
+F 0 "#PWR14" H 8600 2200 30  0001 C CNN
 F 1 "GND" H 8600 2130 30  0001 C CNN
 	1    8600 2200
@@
 $EndComp
 $Comp
-L VCC #PWR013
+L VCC #PWR17
 U 1 1 4F69ED07
 P 9550 950
-F 0 "#PWR013" H 9550 1050 30  0001 C CNN
+F 0 "#PWR17" H 9550 1050 30  0001 C CNN
 F 1 "VCC" H 9550 1050 30  0000 C CNN
 	1    9550 950
@@
 $EndComp
 $Comp
-L GND #PWR014
+L GND #PWR12
 U 1 1 4F69F13E
 P 7800 2200
-F 0 "#PWR014" H 7800 2200 30  0001 C CNN
+F 0 "#PWR12" H 7800 2200 30  0001 C CNN
 F 1 "GND" H 7800 2130 30  0001 C CNN
 	1    7800 2200
@@
 $EndComp
 $Comp
-L GND #PWR015
+L GND #PWR18
 U 1 1 4F69F14B
 P 9550 1550
-F 0 "#PWR015" H 9550 1550 30  0001 C CNN
+F 0 "#PWR18" H 9550 1550 30  0001 C CNN
 F 1 "GND" H 9550 1480 30  0001 C CNN
 	1    9550 1550
@@
 V_LED
 $Comp
-L GND #PWR016
+L GND #PWR11
 U 1 1 4F69FDB8
 P 7100 1750
-F 0 "#PWR016" H 7100 1750 30  0001 C CNN
+F 0 "#PWR11" H 7100 1750 30  0001 C CNN
 F 1 "GND" H 7100 1680 30  0001 C CNN
 	1    7100 1750
@@
 $EndComp
 $Comp
-L GND #PWR017
+L GND #PWR22
 U 1 1 4F6A0000
 P 10200 2000
-F 0 "#PWR017" H 10200 2000 30  0001 C CNN
+F 0 "#PWR22" H 10200 2000 30  0001 C CNN
 F 1 "GND" H 10200 1930 30  0001 C CNN
 	1    10200 2000
@@
 Text Notes 6500 7000 0    60   ~ 0
 ATMega328 \n32 TQFP
-Text Label 7450 2900 0    60   ~ 0
+Text Label 7800 2900 0    60   ~ 0
 12V
 Text Label 7100 1000 0    60   ~ 0
@@
 $EndComp
 $Comp
-L GND #PWR018
+L GND #PWR1
 U 1 1 4F7A113A
 P 1050 2150
-F 0 "#PWR018" H 1050 2150 30  0001 C CNN
+F 0 "#PWR1" H 1050 2150 30  0001 C CNN
 F 1 "GND" H 1050 2080 30  0001 C CNN
 	1    1050 2150
@@
 $EndComp
 $Comp
-L GND #PWR019
+L GND #PWR2
 U 1 1 4F7A127D
 P 1250 2350
-F 0 "#PWR019" H 1250 2350 30  0001 C CNN
+F 0 "#PWR2" H 1250 2350 30  0001 C CNN
 F 1 "GND" H 1250 2280 30  0001 C CNN
 	1    1250 2350
@@
 $EndComp
 $Comp
-L GND #PWR020
+L GND #PWR3
 U 1 1 4F7A1283
 P 1500 2350
-F 0 "#PWR020" H 1500 2350 30  0001 C CNN
+F 0 "#PWR3" H 1500 2350 30  0001 C CNN
 F 1 "GND" H 1500 2280 30  0001 C CNN
 	1    1500 2350
@@
 GND
 $Comp
-L GND #PWR021
+L GND #PWR5
 U 1 1 4F7A1B10
 P 2900 3500
-F 0 "#PWR021" H 2900 3500 30  0001 C CNN
+F 0 "#PWR5" H 2900 3500 30  0001 C CNN
 F 1 "GND" H 2900 3430 30  0001 C CNN
 	1    2900 3500
@@
 $EndComp
 $Comp
-L GND #PWR022
+L GND #PWR4
 U 1 1 4F7A34D5
 P 1900 3250
-F 0 "#PWR022" H 1900 3250 30  0001 C CNN
+F 0 "#PWR4" H 1900 3250 30  0001 C CNN
 F 1 "GND" H 1900 3180 30  0001 C CNN
 	1    1900 3250
@@
 NoConn ~ 3800 2500
 NoConn ~ 2000 3350
+$Comp
+L CONN_3 K1
+U 1 1 4F837AD4
+P 5850 2200
+F 0 "K1" V 5800 2200 50  0000 C CNN
+F 1 "CONN_3" V 5900 2200 40  0000 C CNN
+	1    5850 2200
+	-1   0    0    1
+$EndComp
+Text Notes 6750 4200 0    60   ~ 0
+Arduino Pro Mini Connectors
+Text Notes 5750 2550 0    60   ~ 0
+Sensor Connectors
+Text Label 6200 2300 0    60   ~ 0
+GND
+Text Label 6200 2200 0    60   ~ 0
+VCC
+Text Label 6200 2100 0    60   ~ 0
+D7
 $EndSCHEMATC

Commit message: rearranged European Power Board
Parts:
- removed P1, P2: CONN_6, symbol CONN_6
- added P? (x2): CONN_8, symbol CONN_8
Connections:
- wire segments 140 -> 144

Commit message: Power Board EU BOM added
Parts:
- removed C2: 0.1uF, symbol C
- removed P4, P5: CONN_12, symbol CONN_12
- removed P6: CONN_2, symbol CONN_2
- removed TLC1: TLC5940, symbol TLC5940
- added TLC1: TLC5940-PWP, symbol TLC5940-PWP
- gave numbers to parts that had none: 2
Connections:
- net labels removed: POWER
- no-connect marks 11 -> 12
Other:
- note added: "LED Driver\nPWP 28 package"
- note added: "Sensor Connector"
- note removed: "Arduino Pro Mini Connectors"
- note removed: "Decoupling Cap."
- note removed: "LED Driver\n32QFN"
- note removed: "Sensor Connectors"
- moved on the sheet: C5, C6, C7, C8, C9, D1, D10, D11, D12, D13, D14, D15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
