File: PCB_2x2RBee/2x2RBee.kicad_pcb (KiCad board)
At the start: 2 copper layers, 63.5 x 55.9 mm, 59 parts, among them K1 RELAY, K2 RELAY, K3 RELAY, K4 RELAY, P1 5Vreg, P10 I2C, P12 REL3, P13 REL4, P2 CONN_13X2, P3 IN_18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

Commit message: Adding schematic and gerber files for 2x2RBee board
Parts:
- added U6: LowCurVReg, SOT23-5, F.Cu at (81.7, 85.9)
- added U7: LowCurVReg, SOT23-5, F.Cu at (75.3, 85.9)
- moved R12 38.4 mm to (81.7, 89.3)
- moved R14 14.8 mm to (75.4, 89.3)
- moved D14 10.6 mm to (103.9, 92.3)
- moved D13 9.95 mm to (103.8, 89.5)
- moved R17 2.62 mm to (110.2, 81.9)
- moved U1 0.38 mm to (95.2, 85.7)
- moved R18 0.18 mm to (110.2, 84.3)
- moved U2 0.18 mm to (88.4, 85.7)
- moved R6 0.13 mm to (122.4, 92.5)
Connections:
- P1 pad 3: (no net) -> GND
Routing:
- net GND: track 0.00 -> 342.4 mm, vias 0 -> 3
- net /3V3: track 0.00 -> 110.7 mm, vias 0 -> 4
- net /5V-RPI: track 0.00 -> 107.8 mm, vias 0 -> 9
- net /GPIO_4: track 0.00 -> 56.7 mm, vias 0 -> 1
- net /5V-Relay4: track 0.00 -> 46.9 mm
- net /GPIO_17: track 0.00 -> 46.4 mm, vias 0 -> 1
- net /5V-Relay3: track 0.00 -> 38.2 mm
- net /GPIO_23: track 0.00 -> 37.0 mm, vias 0 -> 1
- net /5Vreg: track 0.00 -> 37.0 mm, vias 0 -> 1
- net /5V-Relay2: track 0.00 -> 28.7 mm
- net /GPIO_24: track 0.00 -> 27.5 mm, vias 0 -> 1
- net /MOSI: track 0.00 -> 26.3 mm, vias 0 -> 1
- net /MISO: track 0.00 -> 24.3 mm, vias 0 -> 1
- net /Din: track 0.00 -> 23.1 mm, vias 0 -> 1
- net /SCLK: track 0.00 -> 23.0 mm, vias 0 -> 1
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